File: schematics/bikePov.kicad_pcb (KiCad board)
At the start: 2 copper layers, 98.5 x 57.9 mm, 32 parts, among them J1 WS2812 out, J2 WS2812 in, J3 Micro usb, J4 WS2812 out, J5 WS2812 out, SW1 Power switch, U1 S09, U2 ATtiny85-20PU, U3 Hall sensor

Commit message: changed to camel case and updated PCB
Connections:
- BT1 pad 2: /GND_in -> Net-(BT1-Pad2)
- BT2 pad 2: /GND_in -> Net-(BT1-Pad2)
- U1 pad 3: /GND_in -> Net-(BT1-Pad2)
Routing:
- net /GND_in: track 107.2 -> 39.7 mm
- net Net-(BT1-Pad2): track 0.00 -> 41.4 mm
- removed copper zone on F.Cu, net /GND_in
Other:
- outline, holes or cut-outs redrawn
